Commit message: add r 85 specified module

File: robotiq_85_description/urdf/robotiq_85_gripper.transmission.xacro (robot description, xacro)
@@ -12,37 +12,4 @@
             </actuator>
         </transmission>
-        <gazebo>
-                <!-- loading plugin: mimic joints works in gazebo now -->
-            <plugin filename="libroboticsgroup_gazebo_mimic_joint_plugin.so" name="${prefix}mimic_robotiq_85_1">
-                <joint>${prefix}robotiq_85_left_knuckle_joint</joint>
-                <mimicJoint>${prefix}robotiq_85_right_knuckle_joint</mimicJoint>
-                <!--multiplier>1.0</multiplier>
-                <offset>0.0</offset-->
-            </plugin>
-            <plugin filename="libroboticsgroup_gazebo_mimic_joint_plugin.so" name="${prefix}mimic_robotiq_85_2">
-                <joint>${prefix}robotiq_85_left_knuckle_joint</joint>
-                <mimicJoint>${prefix}robotiq_85_left_inner_knuckle_joint</mimicJoint>
-                <!--multiplier>1.0</multiplier>
-                <offset>0.0</offset-->
-            </plugin>
-            <plugin filename="libroboticsgroup_gazebo_mimic_joint_plugin.so" name="${prefix}mimic_robotiq_85_3">
-                <joint>${prefix}robotiq_85_left_knuckle_joint</joint>
-                <mimicJoint>${prefix}robotiq_85_right_inner_knuckle_joint</mimicJoint>
-                <!--multiplier>1.0</multiplier>
-                <offset>0.0</offset-->
-            </plugin>
-            <plugin filename="libroboticsgroup_gazebo_mimic_joint_plugin.so" name="${prefix}mimic_robotiq_85_4">
-                <joint>${prefix}robotiq_85_left_knuckle_joint</joint>
-                <mimicJoint>${prefix}robotiq_85_left_finger_tip_joint</mimicJoint>
-                <!--multiplier>-1.0</multiplier-->
-                <!--offset>0.0</offset-->
-            </plugin>
-            <plugin filename="libroboticsgroup_gazebo_mimic_joint_plugin.so" name="${prefix}mimic_robotiq_85_5">
-                <joint>${prefix}robotiq_85_left_knuckle_joint</joint>
-                <mimicJoint>${prefix}robotiq_85_right_finger_tip_joint</mimicJoint>
-                <!--multiplier>-1.0</multiplier-->
-                <!--offset>0.0</offset-->
-            </plugin>
-        </gazebo>
     </xacro:macro>
 </robot>
